File: kicad/ESP32_TFT2-8/ESP32_TFT2-8.kicad_pcb (KiCad board)
At the start: 2 copper layers, 144.8 x 73.7 mm, 16 parts, among them U1 ESP32-DevKitC, U10 GAIN, U11 DIN, U12 BCLK, U13 LRC, U14 L+, U15 L-, U3 5V+, U4 GND, U5 Se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

Commit message: V 10092024
Parts:
- removed the G*** at (95.1, 141.1)
- removed U14: L+, !Goody:LP
- removed U15: L-, !Goody:LP
- added G***: LOGO, !Goody:ob-logo_B.SilkS, F.Cu at (192.7, 124.0)
- U10, U11, U12, U13, U7, U8, U9: moved to B.Cu
- moved U3 9.03 mm to (97.9, 93.9)
- moved U4 9.03 mm to (103.0, 93.9)
- moved U5 9.03 mm to (108.1, 93.9)
- moved U6 9.03 mm to (113.2, 93.9)
- moved U11 6.65 mm to (96.8, 117.3)
- moved U13 6.65 mm to (96.8, 122.4)
- moved U7 6.65 mm to (96.8, 107.2)
- moved U8 6.65 mm to (96.8, 109.7)
- moved U9 6.65 mm to (96.8, 112.3)
- moved U10 6.65 mm to (96.8, 114.8)
- moved U12 6.65 mm to (96.8, 119.9)
Connections:
- U2 pad 5: unconnected-(U2-DC-Pad5) -> unconnected-(U1-ADC2_CH0/GPIO4-Pad26)
- U2 pad 8: unconnected-(U2-LED-Pad8) -> Net-(U1-3V3)
Routing:
- net Net-(U10-LP): track 257.8 -> 310.5 mm
- net Net-(U1-5V): track 168.4 -> 123.9 mm
- net unconnected-(U1-ADC2_CH0/GPIO4-Pad26): track 0.00 -> 41.8 mm
- net Net-(U1-3V3): track 136.0 -> 172.2 mm, vias 0 -> 1
- net Net-(U1-32K_XN/GPIO33/ADC1_CH5): track 63.4 -> 70.8 mm
- net Net-(U1-DAC_2/ADC2_CH9/GPIO26): track 69.5 -> 77.0 mm
- net Net-(U1-DAC_1/ADC2_CH8/GPIO25): track 68.1 -> 75.5 mm
- net Net-(U1-ADC2_CH7/GPIO27): track 42.1 -> 46.6 mm
- net unconnected-(U1-CMD-Pad18): track 0.00 -> 4.49 mm
- net unconnected-(U1-SENSOR_VN/GPIO39/ADC1_CH3-Pad4): track 0.00 -> 4.49 mm
- net Net-(U1-MTMS/GPIO14/ADC2_CH6): track 38.9 -> 43.4 mm
- net unconnected-(U1-VDET_2/GPIO35/ADC1_CH7-Pad6): track 0.00 -> 4.49 mm
- net unconnected-(U1-SD_DATA3/GPIO10-Pad17): track 0.00 -> 4.49 mm
- net unconnected-(U1-SD_DATA2/GPIO9-Pad16): track 0.00 -> 4.49 mm
- net unconnected-(U1-MTDI/GPIO12/ADC2_CH5-Pad13): track 0.00 -> 4.49 mm
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Other:
- board size 144.8 x 73.7 mm -> 131.4 x 73.7 mm
- board text added: "BCLK"
- board text added: "CS"
- board text added: "D/C"
- board text added: "DIN"
- board text added: "GAIN"
- board text added: "GND"
- board text added: "KHF 09.2024"
- board text added: "LED"
- board text added: "LRC"
- board text added: "MAX98357"
- board text added: "RESET"
- board text added: "SCK"
- board text added: "SD"
- board text added: "SDI (MOSI)"
- board text added: "SDO (MISO)"
- board text added: "TOUCH"
- board text added: "T_CLK"
- board text added: "T_CS"
- board text added: "T_DIN"
- board text added: "T_DO"
- board text added: "T_IRQ"
- board text added: "VCC"
- board text added: "Vin"
- board text added: "WEB-Radiowecker"
- board text removed: "KHF 07.2024"
- board text removed: "Max98357"
- board text removed: "Radiowecker"

Commit message: V 02102024
Parts:
- moved U13 33.4 mm to (122.0, 100.5), turned to -90 degrees
- moved U12 30.3 mm to (122.0, 103.1), turned to -90 degrees
- moved U11 27.8 mm to (122.0, 105.6), turned to -90 degrees
- moved U7 26.6 mm to (122.0, 115.8), turned to -90 degrees
- moved U10 26.1 mm to (122.0, 108.2), turned to -90 degrees
- moved U8 25.4 mm to (122.0, 113.2), turned to -90 degrees
- moved U9 25.2 mm to (122.0, 110.7), turned to -90 degrees
- moved U3 24.3 mm to (117.4, 79.3)
- moved U4 24.3 mm to (122.4, 79.3)
- moved U5 24.3 mm to (127.5, 79.3)
- moved U6 24.3 mm to (132.6, 79.3)
Routing:
- net Net-(U10-LP): track 310.5 -> 234.8 mm
- net Net-(U1-DAC_1/ADC2_CH8/GPIO25): track 75.5 -> 42.3 mm
- net Net-(U1-3V3): track 172.2 -> 140.6 mm
- net Net-(U1-DAC_2/ADC2_CH9/GPIO26): track 77.0 -> 47.3 mm
- net Net-(U1-32K_XN/GPIO33/ADC1_CH5): track 70.8 -> 44.7 mm
- net Net-(U1-GPIO23): track 146.2 -> 130.9 mm
- net Net-(U1-GPIO18): track 75.3 -> 63.3 mm
- net Net-(U1-5V): track 123.9 -> 116.3 mm
- net Net-(U3-LP): track 20.3 -> 13.7 mm
Other:
- board size 131.4 x 73.7 mm -> 111.2 x 73.7 mm
- board text added: "KHF 10.2024"
- board text removed: "KHF 09.2024"
